Commit message: Added LFS and began to write skeleton tracker class

File: src/panda_world/models/panda/panda_fr3_no_table.urdf (robot description, URDF)
Before this commit: robot fr3, 8 links, 7 joints
Links:
- added link fr3_link8
Joints:
- added joint fr3_joint8: type fixed, parent fr3_link7, child fr3_link8, origin xyz=0 0 0.107 rpy=0 0 0
