Commit message: Implemented almost all the demo for the project
Missing force feedback in impedance controller and review for real
scenario

File: src/panda_world/models/camera.urdf (robot description, URDF)
Before this commit: robot camera, 2 links, 1 joints
Links:
- removed link camera_link
- added link kinect_depth
- added link kinect_rgb, mass 0.1; collision box size=0.05 0.05 0.05; visual box size=0.05 0.05 0.05
Joints:
- added joint camera_depth_joint: type fixed, parent kinect_rgb, child kinect_depth, origin xyz=0 0 0 rpy=0 0 0
- joint camera_joint: child camera_link -> kinect_rgb; origin xyz=0 1.5 3.2 rpy=0.1 0.9 -1.57 -> xyz=0 2.5 3.2 rpy=0.1 0.9 -1.57
